File: cat_tracker.sch (KiCad schematic (older format))
At the start: 32 parts

Commit message: 2021-08-10
Parts:
- D1: renamed from D?; footprint (none) -> Diode_SMD:D_SMA_Handsoldering
- gave numbers to parts that had none: 31

Commit message: 2021-08-10 2
Parts:
- C1, C10, C11, C2, C3, C4, C5, C6, C7, C8, C9: symbol Device:C -> cat_tracker-rescue:C-Device
- D1: symbol Device:D_Schottky -> cat_tracker-rescue:D_Schottky-Device
- D2: symbol Device:LED -> cat_tracker-rescue:LED-Device
- J1: symbol Connector_Generic:Conn_01x02 -> cat_tracker-rescue:Conn_01x02-Connector_Generic
- J2: symbol Connector_Generic:Conn_01x04 -> cat_tracker-rescue:Conn_01x04-Connector_Generic
- R1, R10, R2, R3, R4, R5, R6, R7, R8, R9: symbol Device:R -> cat_tracker-rescue:R-Device
- SW1, SW2: symbol Switch:SW_Push -> cat_tracker-rescue:SW_Push-Switch
- U3: symbol Battery_Management:MCP73831-2-OT -> cat_tracker-rescue:MCP73831-2-OT-Battery_Management
- U4: symbol RF_Module:ESP32-WROOM-32D -> cat_tracker-rescue:ESP32-WROOM-32D-RF_Module
- U5: symbol Sensor_Motion:MPU-6050 -> cat_tracker-rescue:MPU-6050-Sensor_Motion
Changed lines of the file:
@@
 $EndDescr
 $Comp
-L RF_Module:ESP32-WROOM-32D U4
+L cat_tracker-rescue:ESP32-WROOM-32D-RF_Module U4
 U 1 1 61108DF0
 P 5550 4500
@@
 $EndComp
 $Comp
-L Battery_Management:MCP73831-2-OT U3
+L cat_tracker-rescue:MCP73831-2-OT-Battery_Management U3
 U 1 1 6110E339
 P 4800 1500
@@
 $EndComp
 $Comp
-L Device:D_Schottky D1
+L cat_tracker-rescue:D_Schottky-Device D1
 U 1 1 611100B7
 P 4550 1000
@@
 $EndComp
 $Comp
-L Device:C C1
+L cat_tracker-rescue:C-Device C1
 U 1 1 6111090E
 P 2700 1500
@@
 $EndComp
 $Comp
-L Device:C C2
+L cat_tracker-rescue:C-Device C2
 U 1 1 61112178
 P 3150 1500
@@
 	2350 1650 2250 1650
 $Comp
-L power:Earth #PWR0101
+L cat_tracker-rescue:Earth-power #PWR0101
 U 1 1 61112600
 P 2250 1750
@@
 $EndComp
 $Comp
-L power:Earth #PWR0102
+L cat_tracker-rescue:Earth-power #PWR0102
 U 1 1 6111274F
 P 2250 1250
@@
 $EndComp
 $Comp
-L power:Earth #PWR0103
+L cat_tracker-rescue:Earth-power #PWR0103
 U 1 1 61112BC4
 P 2700 1650
@@
 $EndComp
 $Comp
-L power:Earth #PWR0104
+L cat_tracker-rescue:Earth-power #PWR0104
 U 1 1 611130BC
 P 3150 1650
@@
 VBUS
 $Comp
-L Device:LED D2
+L cat_tracker-rescue:LED-Device D2
 U 1 1 61114FC1
 P 5050 1000
@@
 $EndComp
 $Comp
-L Device:R R1
+L cat_tracker-rescue:R-Device R1
 U 1 1 61115A90
 P 5400 1150
@@
 $EndComp
 $Comp
-L Device:R R3
+L cat_tracker-rescue:R-Device R3
 U 1 1 6111654E
 P 4300 1750
@@
 $EndComp
 $Comp
-L Device:C C5
+L cat_tracker-rescue:C-Device C5
 U 1 1 61116BD2
 P 5650 1550
@@
 $EndComp
 $Comp
-L power:Earth #PWR0105
+L cat_tracker-rescue:Earth-power #PWR0105
 U 1 1 611173E7
 P 4300 1900
@@
 $EndComp
 $Comp
-L power:Earth #PWR0106
+L cat_tracker-rescue:Earth-power #PWR0106
 U 1 1 6111791D
 P 4800 1800
@@
 	5200 1400 5650 1400
 $Comp
-L power:Earth #PWR0107
+L cat_tracker-rescue:Earth-power #PWR0107
 U 1 1 61118BDB
 P 5650 1700
@@
 	4300 1600 4400 1600
 $Comp
-L Connector_Generic:Conn_01x02 J1
+L cat_tracker-rescue:Conn_01x02-Connector_Generic J1
 U 1 1 6111965B
 P 6300 1400
@@
 $EndComp
 $Comp
-L power:Earth #PWR0108
+L cat_tracker-rescue:Earth-power #PWR0108
 U 1 1 61119EBD
 P 6000 1600
@@
 $EndComp
 $Comp
-L Device:C C3
+L cat_tracker-rescue:C-Device C3
 U 1 1 6111DBE3
 P 7300 1500
@@
 	7650 1350 7750 1350
 $Comp
-L power:Earth #PWR0109
+L cat_tracker-rescue:Earth-power #PWR0109
 U 1 1 6111EF7B
 P 7300 1650
@@
 $EndComp
 $Comp
-L power:Earth #PWR0110
+L cat_tracker-rescue:Earth-power #PWR0110
 U 1 1 6111F802
 P 7650 1650
@@
 	7650 1550 7750 1550
 $Comp
-L Device:R R2
+L cat_tracker-rescue:R-Device R2
 U 1 1 61120B43
 P 8650 1500
@@
 	8450 1550 8350 1550
 $Comp
-L power:+3.3V #PWR0111
+L cat_tracker-rescue:+3.3V-power #PWR0111
 U 1 1 611226CB
 P 8950 1350
@@
 $EndComp
 $Comp
-L Device:C C4
+L cat_tracker-rescue:C-Device C4
 U 1 1 61123213
 P 8950 1500
@@
 Connection ~ 8650 1350
 $Comp
-L power:Earth #PWR0112
+L cat_tracker-rescue:Earth-power #PWR0112
 U 1 1 611243DC
 P 8950 1650
@@
 $EndComp
 $Comp
-L power:+3.3V #PWR0113
+L cat_tracker-rescue:+3.3V-power #PWR0113
 U 1 1 61124907
 P 5550 3100
@@
 EN
 $Comp
-L power:Earth #PWR0114
+L cat_tracker-rescue:Earth-power #PWR0114
 U 1 1 61126409
 P 5550 5900
@@
 SCL
 $Comp
-L Sensor_Motion:MPU-6050 U5
+L cat_tracker-rescue:MPU-6050-Sensor_Motion U5
 U 1 1 61129188
 P 8950 4800
@@
 $EndComp
 $Comp
-L Device:C C10
+L cat_tracker-rescue:C-Device C10
 U 1 1 6112A116
 P 9750 5350
@@
 	9750 5100 9650 5100
 $Comp
-L power:Earth #PWR0115
+L cat_tracker-rescue:Earth-power #PWR0115
 U 1 1 6112E17E
 P 9750 5500
@@
 $EndComp
 $Comp
-L Device:C C11
+L cat_tracker-rescue:C-Device C11
 U 1 1 6112EAEE
 P 9950 5350
@@
 	9950 5000 9950 5200
 $Comp
-L power:Earth #PWR0116
+L cat_tracker-rescue:Earth-power #PWR0116
 U 1 1 611305F1
 P 9950 5500
@@
 $EndComp
 $Comp
-L power:+3.3V #PWR0117
+L cat_tracker-rescue:+3.3V-power #PWR0117
 U 1 1 611309D0
 P 9050 3900
@@
 	9050 3900 9050 4000
 $Comp
-L Device:C C9
+L cat_tracker-rescue:C-Device C9
 U 1 1 611320D5
 P 9300 4000
@@
 	9050 4000 9050 4100
 $Comp
-L power:Earth #PWR0118
+L cat_tracker-rescue:Earth-power #PWR0118
 U 1 1 61133564
 P 9450 4000
@@
 $EndComp
 $Comp
-L Device:C C8
+L cat_tracker-rescue:C-Device C8
 U 1 1 61134489
 P 8600 4000
@@
 	8850 4000 8850 4100
 $Comp
-L power:+3.3V #PWR0119
+L cat_tracker-rescue:+3.3V-power #PWR0119
 U 1 1 61136FAE
 P 8850 3900
@@
 Connection ~ 8850 4000
 $Comp
-L power:Earth #PWR0120
+L cat_tracker-rescue:Earth-power #PWR0120
 U 1 1 61137FA3
 P 8450 4000
@@
 $EndComp
 $Comp
-L Device:R R7
+L cat_tracker-rescue:R-Device R7
 U 1 1 61138B2F
 P 8150 4250
@@
 	8150 4500 8250 4500
 $Comp
-L Device:R R6
+L cat_tracker-rescue:R-Device R6
 U 1 1 6113BEA6
 P 8050 4250
@@
 $EndComp
 $Comp
-L power:+3.3V #PWR0121
+L cat_tracker-rescue:+3.3V-power #PWR0121
 U 1 1 6113C14C
 P 8050 4100
@@
 	8050 4600 8250 4600
 $Comp
-L Device:R R9
+L cat_tracker-rescue:R-Device R9
 U 1 1 6113DF4F
 P 7800 4700
@@
 $EndComp
 $Comp
-L Device:R R10
+L cat_tracker-rescue:R-Device R10
 U 1 1 6113EEE6
 P 7800 4800
@@
 	7950 4700 8150 4700
 $Comp
-L power:Earth #PWR0122
+L cat_tracker-rescue:Earth-power #PWR0122
 U 1 1 61140E48
 P 7650 4700
@@
 $EndComp
 $Comp
-L power:+3.3V #PWR0123
+L cat_tracker-rescue:+3.3V-power #PWR0123
 U 1 1 61141568
 P 7650 4800
@@
 $EndComp
 $Comp
-L power:Earth #PWR0124
+L cat_tracker-rescue:Earth-power #PWR0124
 U 1 1 61141F59
 P 8250 5000
@@
 $EndComp
 $Comp
-L power:Earth #PWR0125
+L cat_tracker-rescue:Earth-power #PWR0125
 U 1 1 61142530
 P 8250 5100
@@
 INT
 $Comp
-L Device:R R8
+L cat_tracker-rescue:R-Device R8
 U 1 1 61147981
 P 9750 4250
@@
 $EndComp
 $Comp
-L power:+3.3V #PWR0126
+L cat_tracker-rescue:+3.3V-power #PWR0126
 U 1 1 611481E3
 P 9750 4100
@@
 Connection ~ 9750 4500
 $Comp
-L power:Earth #PWR0127
+L cat_tracker-rescue:Earth-power #PWR0127
 U 1 1 6114AF17
 P 8950 5500
@@
 INT
 $Comp
-L Switch:SW_Push SW1
+L cat_tracker-rescue:SW_Push-Switch SW1
 U 1 1 6115F88F
 P 1600 3300
@@
 $EndComp
 $Comp
-L power:+3.3V #PWR0128
+L cat_tracker-rescue:+3.3V-power #PWR0128
 U 1 1 6115FA35
 P 1300 3200
@@
 	1300 3300 1400 3300
 $Comp
-L Connector_Generic:Conn_01x04 J2
+L cat_tracker-rescue:Conn_01x04-Connector_Generic J2
 U 1 1 611619C1
 P 1600 4450
@@
 $EndComp
 $Comp
-L power:+3.3V #PWR0129
+L cat_tracker-rescue:+3.3V-power #PWR0129
 U 1 1 61162905
 P 1800 4350
@@
 $EndComp
 $Comp
-L power:Earth #PWR0130
+L cat_tracker-rescue:Earth-power #PWR0130
 U 1 1 611632DD
 P 1800 4450
@@
 TX
 $Comp
-L Device:C C6
+L cat_tracker-rescue:C-Device C6
 U 1 1 6116473C
 P 1800 3450
@@
 $EndComp
 $Comp
-L Device:R R4
+L cat_tracker-rescue:R-Device R4
 U 1 1 61164D5E
 P 1950 3300
@@
 Connection ~ 1800 3300
 $Comp
-L power:Earth #PWR0131
+L cat_tracker-rescue:Earth-power #PWR0131
 U 1 1 611655D5
 P 1800 3600
@@
 BOOT
 $Comp
-L Switch:SW_Push SW2
+L cat_tracker-rescue:SW_Push-Switch SW2
 U 1 1 6116806C
 P 2800 3300
@@
 $EndComp
 $Comp
-L power:+3.3V #PWR0132
+L cat_tracker-rescue:+3.3V-power #PWR0132
 U 1 1 61168072
 P 2500 3200
@@
 	2500 3300 2600 3300
 $Comp
-L Device:C C7
+L cat_tracker-rescue:C-Device C7
 U 1 1 6116807A
 P 3000 3450
@@
 $EndComp
 $Comp
-L Device:R R5
+L cat_tracker-rescue:R-Device R5
 U 1 1 61168080
 P 3150 3300
@@
 Connection ~ 3000 3300
 $Comp
-L power:Earth #PWR0133
+L cat_tracker-rescue:Earth-power #PWR0133
 U 1 1 61168087
 P 3000 3600

Commit message: 2021-08-29
Connections:
- net SCL: no longer U4.33 (IO21)
- net SDA: now reaches R7.1, U5.24 (SDA)
- net SDA: now also U4.33 (IO21)
Changed lines of the file:
@@
 	-1   0    0    1
 $EndComp
-Wire Wire Line
-	8150 4400 8150 4500
-Wire Wire Line
-	8150 4500 8250 4500
 $Comp
 L cat_tracker-rescue:R-Device R6
@@
 	8050 4100 8150 4100
 Connection ~ 8050 4100
-Wire Wire Line
-	8050 4400 8050 4500
-Wire Wire Line
-	8050 4600 8250 4600
 $Comp
 L cat_tracker-rescue:R-Device R9
@@
 Text GLabel 7900 4600 0    50   Input ~ 0
 SCL
-Wire Wire Line
-	7900 4600 8050 4600
-Connection ~ 8050 4600
-Wire Wire Line
-	7900 4500 8050 4500
-Connection ~ 8050 4500
-Wire Wire Line
-	8050 4500 8050 4600
 Text GLabel 9850 4500 2    50   Input ~ 0
 INT
@@
 Text GLabel 3300 3300 2    50   Input ~ 0
 BOOT
+Wire Wire Line
+	7900 4500 8150 4500
+Wire Wire Line
+	7900 4600 8050 4600
+Wire Wire Line
+	8050 4400 8050 4600
+Connection ~ 8050 4600
+Wire Wire Line
+	8050 4600 8250 4600
+Wire Wire Line
+	8150 4400 8150 4500
+Connection ~ 8150 4500
+Wire Wire Line
+	8150 4500 8250 4500
 $EndSCHEMATC

Commit message: 2021-08-30
Parts:
- removed D1: SK24/SMA, Diode_SMD:D_SMA_Handsoldering, symbol cat_tracker-rescue:D_Schottky-Device
- removed R2: 100k, Resistor_SMD:R_0603_1608Metric_Pad0.98x0.95mm_HandSolder, symbol cat_tracker-rescue:R-Device
- removed U1: NCP187, Package_DFN_QFN:DFN-6-1EP_2x2mm_P0.65mm_EP1x1.6mm, symbol add_LDO:NCP187
- added C13: 100n, Capacitor_SMD:C_0603_1608Metric_Pad1.08x0.95mm_HandSolder, symbol cat_tracker-rescue:C-Device
- added C6: 0.01u, Capacitor_SMD:C_0603_1608Metric_Pad1.08x0.95mm_HandSolder, symbol cat_tracker-rescue:C-Device
- added D2: LED/2012, LED_SMD:LED_0805_2012Metric_Pad1.15x1.40mm_HandSolder, symbol cat_tracker-rescue:LED-Device
- added R12: 1k, Resistor_SMD:R_0603_1608Metric_Pad0.98x0.95mm_HandSolder, symbol cat_tracker-rescue:R-Device
- added R13: 510, Resistor_SMD:R_0603_1608Metric_Pad0.98x0.95mm_HandSolder, symbol cat_tracker-rescue:R-Device
- added R3, R4: 100k, Resistor_SMD:R_0603_1608Metric_Pad0.98x0.95mm_HandSolder, symbol cat_tracker-rescue:R-Device
- added SW3: EN Btn, ali_Switch:NW3-A03-05, symbol cat_tracker-rescue:SW_Push-Switch
- added U1: MIC5318-3.3YD5-TR, Package_TO_SOT_SMD:SOT-23-5, symbol MIC531833YD5TR:MIC5318-3.3YD5-TR
- C4: value 10u -> 0.1u
- R5: renamed from R4; value 1k -> 100
- renumbered C9 to C10, C10 to C11, C11 to C12, C6 to C7, C7 to C8, C8 to C9, D2 to D1, R9 to R10, R10 to R11, R3 to R2, R5 to R6, R6 to R7, R7 to R8, R8 to R9
Connections:
- net +3V3: now also R3.2, R4.2, SW3.1, U1.5 (OUT); no longer SW1.1, SW2.1
- net BATT: now also U1.1 (IN), U1.3 (EN)
- net BOOT: now also R4.1
- net EN: now also R3.1
- net Earth: now also SW1.1, SW2.1, C13.2, C6.2, R13.1, U1.2 (GND)
- net VBUS: now also D1.2 (A), U3.4 (VDD)
- net CHRG: now reaches U4.28 (IO17)
- net CHRG: now also R1.2, U3.1 (STAT)
- net BTN: now reaches U4.30 (IO18)
- net BTN: now also R12.1
- net LED: now reaches U4.31 (IO19)
- net LED: now also D2.2 (A)
- new net: C6.1, U1.4 (BYP)
- new net: C13.1, R12.2, SW3.2
- new net: D2.1 (K), R13.2
Other:
- moved on the sheet: C3, C4

Commit message: 2021-09-17
Parts:
- removed C8: 100n, Capacitor_SMD:C_0603_1608Metric_Pad1.08x0.95mm_HandSolder, symbol cat_tracker-rescue:C-Device
- removed R3, R4: 100k, Resistor_SMD:R_0603_1608Metric_Pad0.98x0.95mm_HandSolder, symbol cat_tracker-rescue:R-Device
- removed R6: 1k, Resistor_SMD:R_0603_1608Metric_Pad0.98x0.95mm_HandSolder, symbol cat_tracker-rescue:R-Device
- removed SW2: EN Btn, ali_Switch:NW3-A03-05, symbol cat_tracker-rescue:SW_Push-Switch
- added TP?: TestPoint_2Pole, symbol Connector:TestPoint_2Pole
- C7: value 100n -> 1u
- R5: value 100 -> 10k
- SW3: value EN Btn -> Btn
Connections:
- net BOOT: now also TP?.2
- net Earth: now also TP?.1
Changed lines of the file:
@@
 P 1800 3450
 F 0 "C7" H 1915 3496 50  0000 L CNN
-F 1 "100n" H 1915 3405 50  0000 L CNN
+F 1 "1u" H 1915 3405 50  0000 L CNN
 F 2 "Capacitor_SMD:C_0603_1608Metric_Pad1.08x0.95mm_HandSolder" H 1838 3300 50  0001 C CNN
 F 3 "~" H 1800 3450 50  0001 C CNN
@@
 P 1950 3300
 F 0 "R5" V 1850 3250 50  0000 L CNN
-F 1 "100" V 1950 3300 50  0000 C CNN
+F 1 "10k" V 1950 3300 50  0000 C CNN
 F 2 "Resistor_SMD:R_0603_1608Metric_Pad0.98x0.95mm_HandSolder" V 1880 3300 50  0001 C CNN
 F 3 "~" H 1950 3300 50  0001 C CNN
@@
 Text GLabel 6150 3300 2    50   Input ~ 0
 BOOT
-$Comp
-L cat_tracker-rescue:SW_Push-Switch SW2
-U 1 1 6116806C
-P 2800 3300
-F 0 "SW2" H 2800 3585 50  0000 C CNN
-F 1 "EN Btn" H 2800 3494 50  0000 C CNN
-F 2 "ali_Switch:NW3-A03-05" H 2800 3500 50  0001 C CNN
-F 3 "~" H 2800 3500 50  0001 C CNN
-	1    2800 3300
-	1    0    0    -1
-$EndComp
-$Comp
-L cat_tracker-rescue:C-Device C8
-U 1 1 6116807A
-P 3000 3450
-F 0 "C8" H 3115 3496 50  0000 L CNN
-F 1 "100n" H 3115 3405 50  0000 L CNN
-F 2 "Capacitor_SMD:C_0603_1608Metric_Pad1.08x0.95mm_HandSolder" H 3038 3300 50  0001 C CNN
-F 3 "~" H 3000 3450 50  0001 C CNN
-	1    3000 3450
-	1    0    0    -1
-$EndComp
-$Comp
-L cat_tracker-rescue:R-Device R6
-U 1 1 61168080
-P 3150 3300
-F 0 "R6" V 3050 3250 50  0000 L CNN
-F 1 "1k" V 3150 3300 50  0000 C CNN
-F 2 "Resistor_SMD:R_0603_1608Metric_Pad0.98x0.95mm_HandSolder" V 3080 3300 50  0001 C CNN
-F 3 "~" H 3150 3300 50  0001 C CNN
-	1    3150 3300
-	0    1    1    0
-$EndComp
-Connection ~ 3000 3300
-$Comp
-L cat_tracker-rescue:Earth-power #PWR020
-U 1 1 61168087
-P 3000 3600
-F 0 "#PWR020" H 3000 3350 50  0001 C CNN
-F 1 "Earth" H 3000 3450 50  0001 C CNN
-F 2 "" H 3000 3600 50  0001 C CNN
-F 3 "~" H 3000 3600 50  0001 C CNN
-	1    3000 3600
-	1    0    0    -1
-$EndComp
-Text GLabel 3400 3300 2    50   Input ~ 0
-BOOT
 Wire Wire Line
 	7900 4500 8150 4500
@@
 	1    0    0    -1
 $EndComp
-$Comp
-L cat_tracker-rescue:Earth-power #PWR018
-U 1 1 612CA101
-P 2600 3300
-F 0 "#PWR018" H 2600 3050 50  0001 C CNN
-F 1 "Earth" H 2600 3150 50  0001 C CNN
-F 2 "" H 2600 3300 50  0001 C CNN
-F 3 "~" H 2600 3300 50  0001 C CNN
-	1    2600 3300
-	1    0    0    -1
-$EndComp
-$Comp
-L cat_tracker-rescue:R-Device R3
-U 1 1 612CA921
-P 2150 3100
-F 0 "R3" V 2050 3050 50  0000 L CNN
-F 1 "100k" V 2150 3100 50  0000 C CNN
-F 2 "Resistor_SMD:R_0603_1608Metric_Pad0.98x0.95mm_HandSolder" V 2080 3100 50  0001 C CNN
-F 3 "~" H 2150 3100 50  0001 C CNN
-	1    2150 3100
-	-1   0    0    1
-$EndComp
-$Comp
-L cat_tracker-rescue:+3.3V-power #PWR014
-U 1 1 612CB2E7
-P 2150 2950
-F 0 "#PWR014" H 2150 2800 50  0001 C CNN
-F 1 "+3.3V" V 2165 3078 50  0000 L CNN
-F 2 "" H 2150 2950 50  0001 C CNN
-F 3 "" H 2150 2950 50  0001 C CNN
-	1    2150 2950
-	1    0    0    -1
-$EndComp
-$Comp
-L cat_tracker-rescue:R-Device R4
-U 1 1 612CD059
-P 3350 3100
-F 0 "R4" V 3250 3050 50  0000 L CNN
-F 1 "100k" V 3350 3100 50  0000 C CNN
-F 2 "Resistor_SMD:R_0603_1608Metric_Pad0.98x0.95mm_HandSolder" V 3280 3100 50  0001 C CNN
-F 3 "~" H 3350 3100 50  0001 C CNN
-	1    3350 3100
-	-1   0    0    1
-$EndComp
-Wire Wire Line
-	3350 3250 3350 3300
-Wire Wire Line
-	3350 3300 3300 3300
-Wire Wire Line
-	3350 3300 3400 3300
-Connection ~ 3350 3300
-$Comp
-L cat_tracker-rescue:+3.3V-power #PWR015
-U 1 1 612D041F
-P 3350 2950
-F 0 "#PWR015" H 3350 2800 50  0001 C CNN
-F 1 "+3.3V" V 3365 3078 50  0000 L CNN
-F 2 "" H 3350 2950 50  0001 C CNN
-F 3 "" H 3350 2950 50  0001 C CNN
-	1    3350 2950
-	1    0    0    -1
-$EndComp
-Wire Wire Line
-	2200 3300 2150 3300
-Wire Wire Line
-	2150 3250 2150 3300
-Connection ~ 2150 3300
-Wire Wire Line
-	2150 3300 2100 3300
 Wire Wire Line
 	4400 1000 4800 1000
@@
 $EndComp
 $Comp
-L cat_tracker-rescue:SW_Push-Switch SW3
-U 1 1 612E8D33
-P 2350 5650
-F 0 "SW3" H 2350 5935 50  0000 C CNN
-F 1 "EN Btn" H 2350 5844 50  0000 C CNN
-F 2 "ali_Switch:NW3-A03-05" H 2350 5850 50  0001 C CNN
-F 3 "~" H 2350 5850 50  0001 C CNN
-	1    2350 5650
-	1    0    0    -1
-$EndComp
+L cat_tracker-rescue:Earth-power #PWR038
+U 1 1 612EB5D1
+P 2550 5950
+F 0 "#PWR038" H 2550 5700 50  0001 C CNN
+F 1 "Earth" H 2550 5800 50  0001 C CNN
+F 2 "" H 2550 5950 50  0001 C CNN
+F 3 "~" H 2550 5950 50  0001 C CNN
+	1    2550 5950
+	1    0    0    -1
+$EndComp
+Text GLabel 6150 4500 2    50   Input ~ 0
+BTN
+Text GLabel 2850 5650 2    50   Input ~ 0
+BTN
+Text GLabel 6150 4600 2    50   Input ~ 0
+LED
+$Comp
+L cat_tracker-rescue:LED-Device D2
+U 1 1 612ED7C6
+P 2550 6550
+F 0 "D2" H 2543 6295 50  0000 C CNN
+F 1 "LED/2012" H 2543 6386 50  0000 C CNN
+F 2 "LED_SMD:LED_0805_2012Metric_Pad1.15x1.40mm_HandSolder" H 2550 6550 50  0001 C CNN
+F 3 "~" H 2550 6550 50  0001 C CNN
+	1    2550 6550
+	-1   0    0    1
+$EndComp
+$Comp
+L cat_tracker-rescue:R-Device R13
+U 1 1 612EFCE3
+P 2850 6550
+F 0 "R13" V 2750 6500 50  0000 L CNN
+F 1 "510" V 2850 6550 50  0000 C CNN
+F 2 "Resistor_SMD:R_0603_1608Metric_Pad0.98x0.95mm_HandSolder" V 2780 6550 50  0001 C CNN
+F 3 "~" H 2850 6550 50  0001 C CNN
+	1    2850 6550
+	0    1    1    0
+$EndComp
+Text GLabel 2400 6550 0    50   Input ~ 0
+LED
+$Comp
+L cat_tracker-rescue:Earth-power #PWR039
+U 1 1 612F1892
+P 3000 6550
+F 0 "#PWR039" H 3000 6300 50  0001 C CNN
+F 1 "Earth" H 3000 6400 50  0001 C CNN
+F 2 "" H 3000 6550 50  0001 C CNN
+F 3 "~" H 3000 6550 50  0001 C CNN
+	1    3000 6550
+	0    -1   -1   0
+$EndComp
+Text GLabel 5400 1600 3    50   Input ~ 0
+CHRG
+Text GLabel 6150 4400 2    50   Input ~ 0
+CHRG
+Wire Wire Line
+	2100 3300 2200 3300
 $Comp
 L cat_tracker-rescue:C-Device C13
@@
 $EndComp
 $Comp
-L cat_tracker-rescue:Earth-power #PWR038
-U 1 1 612EB5D1
-P 2550 5950
-F 0 "#PWR038" H 2550 5700 50  0001 C CNN
-F 1 "Earth" H 2550 5800 50  0001 C CNN
-F 2 "" H 2550 5950 50  0001 C CNN
-F 3 "~" H 2550 5950 50  0001 C CNN
-	1    2550 5950
-	1    0    0    -1
-$EndComp
+L cat_tracker-rescue:SW_Push-Switch SW3
+U 1 1 612E8D33
+P 2350 5650
+F 0 "SW3" H 2350 5935 50  0000 C CNN
+F 1 "Btn" H 2350 5844 50  0000 C CNN
+F 2 "ali_Switch:NW3-A03-05" H 2350 5850 50  0001 C CNN
+F 3 "~" H 2350 5850 50  0001 C CNN
+	1    2350 5650
+	1    0    0    -1
+$EndComp
+Connection ~ 2550 5650
 $Comp
 L cat_tracker-rescue:R-Device R12
@@
 	0    1    1    0
 $EndComp
-Connection ~ 2550 5650
 $Comp
 L cat_tracker-rescue:+3.3V-power #PWR036
@@
 	1    0    0    -1
 $EndComp
-Text GLabel 6150 4500 2    50   Input ~ 0
-BTN
-Text GLabel 2850 5650 2    50   Input ~ 0
-BTN
-Text GLabel 6150 4600 2    50   Input ~ 0
-LED
-$Comp
-L cat_tracker-rescue:LED-Device D2
-U 1 1 612ED7C6
-P 2550 6550
-F 0 "D2" H 2543 6295 50  0000 C CNN
-F 1 "LED/2012" H 2543 6386 50  0000 C CNN
-F 2 "LED_SMD:LED_0805_2012Metric_Pad1.15x1.40mm_HandSolder" H 2550 6550 50  0001 C CNN
-F 3 "~" H 2550 6550 50  0001 C CNN
-	1    2550 6550
-	-1   0    0    1
-$EndComp
-$Comp
-L cat_tracker-rescue:R-Device R13
-U 1 1 612EFCE3
-P 2850 6550
-F 0 "R13" V 2750 6500 50  0000 L CNN
-F 1 "510" V 2850 6550 50  0000 C CNN
-F 2 "Resistor_SMD:R_0603_1608Metric_Pad0.98x0.95mm_HandSolder" V 2780 6550 50  0001 C CNN
-F 3 "~" H 2850 6550 50  0001 C CNN
-	1    2850 6550
-	0    1    1    0
-$EndComp
-Text GLabel 2400 6550 0    50   Input ~ 0
-LED
-$Comp
-L cat_tracker-rescue:Earth-power #PWR039
-U 1 1 612F1892
-P 3000 6550
-F 0 "#PWR039" H 3000 6300 50  0001 C CNN
-F 1 "Earth" H 3000 6400 50  0001 C CNN
-F 2 "" H 3000 6550 50  0001 C CNN
-F 3 "~" H 3000 6550 50  0001 C CNN
-	1    3000 6550
-	0    -1   -1   0
-$EndComp
-Text GLabel 5400 1600 3    50   Input ~ 0
-CHRG
-Text GLabel 6150 4400 2    50   Input ~ 0
-CHRG
+$Comp
+L Connector:TestPoint_2Pole TP?
+U 1 1 6144C273
+P 2900 3300
+F 0 "TP?" H 2900 3495 50  0000 C CNN
+F 1 "TestPoint_2Pole" H 2900 3404 50  0000 C CNN
+F 2 "" H 2900 3300 50  0001 C CNN
+F 3 "~" H 2900 3300 50  0001 C CNN
+	1    2900 3300
+	1    0    0    -1
+$EndComp
+$Comp
+L cat_tracker-rescue:Earth-power #PWR?
+U 1 1 6144CA62
+P 2700 3300
+F 0 "#PWR?" H 2700 3050 50  0001 C CNN
+F 1 "Earth" H 2700 3150 50  0001 C CNN
+F 2 "" H 2700 3300 50  0001 C CNN
+F 3 "~" H 2700 3300 50  0001 C CNN
+	1    2700 3300
+	1    0    0    -1
+$EndComp
+Text GLabel 3100 3300 2    50   Input ~ 0
+BOOT
 $EndSCHEMATC
